Commit message: Adds the IMU in the robot model and the imu sensor plugin.

File: gpg_description/urdf/gpg.gazebo.xacro (robot description, xacro)
@@ -1,4 +1,7 @@
 <?xml version="1.0"?>
 <robot name="gpg3_sim" xmlns:xacro="http://ros.org/wiki/xacro">
+  <xacro:arg name="laser_visual" default="false"/>
+  <xacro:arg name="imu_visual"   default="true"/>
+  <xacro:arg name="distance_visual" default="false"/>
   <!-- Base_link -->
   <gazebo reference="base_link_cad">
@@ -46,5 +49,5 @@
     </joint>
   </transmission>
-  <!-- Caster back mechanical properties -->
+  <!-- Caster mechanical properties -->
   <gazebo reference="caster_back_link">
     <mu1>0.001</mu1>
@@ -75,4 +78,41 @@
     </joint>
   </transmission>
+  <!-- IMU sensor -->
+  <gazebo reference="imu_link">
+    <sensor type="imu" name="imu">
+      <always_on>true</always_on>
+      <visualize>$(arg imu_visual)</visualize>
+    </sensor>
+    <material>Gazebo/FlatBlack</material>
+  </gazebo>
+  <!-- IMU plugin -->
+  <gazebo>
+    <plugin name="imu_plugin" filename="libgazebo_ros_imu.so">
+      <alwaysOn>true</alwaysOn>
+      <bodyName>imu_link</bodyName>
+      <frameName>imu_link</frameName>
+      <topicName>imu</topicName>
+      <serviceName>imu_service</serviceName>
+      <gaussianNoise>0.0</gaussianNoise>
+      <updateRate>200</updateRate>
+      <imu>
+        <noise>
+          <type>gaussian</type>
+          <rate>
+            <mean>0.0</mean>
+            <stddev>2e-4</stddev>
+            <bias_mean>0.0000075</bias_mean>
+            <bias_stddev>0.0000008</bias_stddev>
+          </rate>
+          <accel>
+            <mean>0.0</mean>
+            <stddev>1.7e-2</stddev>
+            <bias_mean>0.1</bias_mean>
+            <bias_stddev>0.001</bias_stddev>
+          </accel>
+        </noise>
+      </imu>
+    </plugin>
+  </gazebo>
   <!-- Gazebo plugin for ROS Control -->
   <gazebo>

File: gpg_description/urdf/gpg.urdf.xacro (robot description, xacro)
@@ -8,5 +8,5 @@
   <xacro:arg name="distance"   default="false"/>
   <xacro:arg name="lds"        default="false"/>
-<!-- ============ 'base_footprint' is the ground link ===================== -->
+  <!-- ============ 'base_footprint' is the ground link ===================== -->
   <link name="base_footprint"/>
   <joint name="base_joint" type="fixed">

Commit message: Adds the lidar sensor and the respective gazebo plugin.

File: gpg_description/urdf/gpg.gazebo.xacro (robot description, xacro)
@@ -1,5 +1,5 @@
 <?xml version="1.0"?>
 <robot name="gpg3_sim" xmlns:xacro="http://ros.org/wiki/xacro">
-  <xacro:arg name="laser_visual" default="false"/>
+  <xacro:arg name="laser_visual" default="true"/> <!-- rays visible in gazebo -->
   <xacro:arg name="imu_visual"   default="true"/>
   <xacro:arg name="distance_visual" default="false"/>
@@ -84,5 +84,5 @@
       <visualize>$(arg imu_visual)</visualize>
     </sensor>
-    <material>Gazebo/FlatBlack</material>
+    <material>Gazebo/Green</material>
   </gazebo>
   <!-- IMU plugin -->
@@ -115,4 +115,43 @@
     </plugin>
   </gazebo>
+  <!-- Laser Distance Sensor YDLIDAR X4 controller-->
+  <gazebo reference="base_scan">
+    <material>Gazebo/FlatBlack</material>
+    <sensor type="ray" name="lds_lfcd_sensor">
+      <pose>0 0 0 0 0 0</pose>
+      <visualize>$(arg laser_visual)</visualize>
+      <update_rate>40</update_rate>
+      <ray>
+        <scan>
+          <horizontal>
+            <!--samples>360</samples>
+            <resolution>1</resolution-->
+            <samples>500</samples>
+            <resolution>0.72</resolution>
+            <min_angle>-3.1416</min_angle>
+            <max_angle>3.1416</max_angle>
+          </horizontal>
+        </scan>
+        <range>
+          <min>0.2</min>
+          <max>10</max>
+          <resolution>0.015</resolution>
+        </range>
+        <noise>
+          <type>gaussian</type>
+          <!-- Noise parameters based on published spec for YDLIDAR X4
+               is 1.5% at half range 4m (= 60mm, "+-160mm" accuracy at max. range 8m).
+               A mean of 0.0m and stddev of 0.020m will put 99.7% of samples
+               within 0.16m of the true reading. -->
+          <mean>0.0</mean>
+          <stddev>0.01</stddev>
+        </noise>
+      </ray>
+      <plugin name="gazebo_ros_lds_lfcd_controller" filename="libgazebo_ros_laser.so">
+        <topicName>scan</topicName>
+        <frameName>base_scan</frameName>
+      </plugin>
+    </sensor>
+  </gazebo>
   <!-- Gazebo plugin for ROS Control -->
   <gazebo>

File: gpg_description/urdf/gpg.urdf.xacro (robot description, xacro)
@@ -185,5 +185,5 @@
   <!-- (JOINTS) Pi Camera -->
     <joint name="camera_joint" type="revolute">
-      <origin xyz="0.04 0 0.04" rpy="0 0 0"/>
+      <origin xyz="0.065 0 0.0" rpy="0 0 0"/>
       <parent link="base_link"/>
       <child link="camera_link"/>
@@ -244,5 +244,5 @@
       <parent link="base_link"/>
       <child link="base_scan"/>
-      <origin xyz="-0.02 0 0.085" rpy="0 0 -1.57"/>
+      <origin xyz="-0.02 0 0.085" rpy="0 0 0"/>
       <!--LDS** origin xyz="-0.02 0 0.07" rpy="0 0 -1.6"/-->
     </joint>

Commit message: Add Realsense D435 camera to the URDF file. Add gpg_localization package, that publishes the robot ground truth pose. Add gpg_elevation_mapping package, fot grid_map filters.

File: gpg_description/urdf/gpg.gazebo.xacro (robot description, xacro)
@@ -1,7 +1,9 @@
 <?xml version="1.0"?>
 <robot name="gpg3_sim" xmlns:xacro="http://ros.org/wiki/xacro">
+  <xacro:arg name="laser" default="false"/>
+  <xacro:arg name="d435"  default="false"/>
+  <xacro:arg name="imu"   default="false"/>
+  <xacro:arg name="imu_visual" default="true"/>
   <xacro:arg name="laser_visual" default="true"/> <!-- rays visible in gazebo -->
-  <xacro:arg name="imu_visual"   default="true"/>
-  <xacro:arg name="distance_visual" default="false"/>
   <!-- Base_link -->
   <gazebo reference="base_link_cad">
@@ -79,79 +81,97 @@
   </transmission>
   <!-- IMU sensor -->
-  <gazebo reference="imu_link">
-    <sensor type="imu" name="imu">
-      <always_on>true</always_on>
-      <visualize>$(arg imu_visual)</visualize>
-    </sensor>
-    <material>Gazebo/Green</material>
-  </gazebo>
-  <!-- IMU plugin -->
-  <gazebo>
-    <plugin name="imu_plugin" filename="libgazebo_ros_imu.so">
-      <alwaysOn>true</alwaysOn>
-      <bodyName>imu_link</bodyName>
-      <frameName>imu_link</frameName>
-      <topicName>imu</topicName>
-      <serviceName>imu_service</serviceName>
-      <gaussianNoise>0.0</gaussianNoise>
-      <updateRate>200</updateRate>
-      <imu>
-        <noise>
-          <type>gaussian</type>
-          <rate>
-            <mean>0.0</mean>
-            <stddev>2e-4</stddev>
-            <bias_mean>0.0000075</bias_mean>
-            <bias_stddev>0.0000008</bias_stddev>
-          </rate>
-          <accel>
-            <mean>0.0</mean>
-            <stddev>1.7e-2</stddev>
-            <bias_mean>0.1</bias_mean>
-            <bias_stddev>0.001</bias_stddev>
-          </accel>
-        </noise>
-      </imu>
-    </plugin>
-  </gazebo>
+  <xacro:if value="$(arg imu)">
+		<gazebo reference="imu_link">
+		  <sensor type="imu" name="imu">
+		    <always_on>true</always_on>
+		    <visualize>$(arg imu_visual)</visualize>
+		  </sensor>
+		  <material>Gazebo/Green</material>
+		</gazebo>
+		<!-- IMU plugin -->
+		<gazebo>
+		  <plugin name="imu_plugin" filename="libgazebo_ros_imu.so">
+		    <alwaysOn>true</alwaysOn>
+		    <bodyName>imu_link</bodyName>
+		    <frameName>imu_link</frameName>
+		    <topicName>imu</topicName>
+		    <serviceName>imu_service</serviceName>
+		    <gaussianNoise>0.0</gaussianNoise>
+		    <updateRate>200</updateRate>
+		    <imu>
+		      <noise>
+		        <type>gaussian</type>
+		        <rate>
+		          <mean>0.0</mean>
+		          <stddev>2e-4</stddev>
+		          <bias_mean>0.0000075</bias_mean>
+		          <bias_stddev>0.0000008</bias_stddev>
+		        </rate>
+		        <accel>
+		          <mean>0.0</mean>
+		          <stddev>1.7e-2</stddev>
+		          <bias_mean>0.1</bias_mean>
+		          <bias_stddev>0.001</bias_stddev>
+		        </accel>
+		      </noise>
+		    </imu>
+		  </plugin>
+		</gazebo>
+  </xacro:if>
   <!-- Laser Distance Sensor YDLIDAR X4 controller-->
-  <gazebo reference="base_scan">
-    <material>Gazebo/FlatBlack</material>
-    <sensor type="ray" name="lds_lfcd_sensor">
-      <pose>0 0 0 0 0 0</pose>
-      <visualize>$(arg laser_visual)</visualize>
-      <update_rate>40</update_rate>
-      <ray>
-        <scan>
-          <horizontal>
-            <!--samples>360</samples>
-            <resolution>1</resolution-->
-            <samples>500</samples>
-            <resolution>0.72</resolution>
-            <min_angle>-3.1416</min_angle>
-            <max_angle>3.1416</max_angle>
-          </horizontal>
-        </scan>
-        <range>
-          <min>0.2</min>
-          <max>10</max>
-          <resolution>0.015</resolution>
-        </range>
-        <noise>
-          <type>gaussian</type>
-          <!-- Noise parameters based on published spec for YDLIDAR X4
-               is 1.5% at half range 4m (= 60mm, "+-160mm" accuracy at max. range 8m).
-               A mean of 0.0m and stddev of 0.020m will put 99.7% of samples
-               within 0.16m of the true reading. -->
-          <mean>0.0</mean>
-          <stddev>0.01</stddev>
-        </noise>
-      </ray>
-      <plugin name="gazebo_ros_lds_lfcd_controller" filename="libgazebo_ros_laser.so">
-        <topicName>scan</topicName>
-        <frameName>base_scan</frameName>
-      </plugin>
-    </sensor>
-  </gazebo>
+  <xacro:if value="$(arg laser)">
+	  <gazebo reference="base_scan">
+			<material>Gazebo/FlatBlack</material>
+			<sensor type="ray" name="lds_lfcd_sensor">
+				<pose>0 0 0 0 0 0</pose>
+				<visualize>$(arg laser_visual)</visualize>
+				<update_rate>40</update_rate>
+				<ray>
+				  <scan>
+				    <horizontal>
+				      <!--samples>360</samples>
+				      <resolution>1</resolution-->
+				      <samples>500</samples>
+				      <resolution>0.72</resolution>
+				      <min_angle>-3.1416</min_angle>
+				      <max_angle>3.1416</max_angle>
+				    </horizontal>
+				  </scan>
+				  <range>
+				    <min>0.2</min>
+				    <max>10</max>
+				    <resolution>0.015</resolution>
+				  </range>
+				  <noise>
+				    <type>gaussian</type>
+				    <!-- Noise parameters based on published spec for YDLIDAR X4
+				         is 1.5% at half range 4m (= 60mm, "+-160mm" accuracy at max. range 8m).
+				         A mean of 0.0m and stddev of 0.020m will put 99.7% of samples
+				         within 0.16m of the true reading. -->
+				    <mean>0.0</mean>
+				    <stddev>0.01</stddev>
+				  </noise>
+				</ray>
+				<plugin name="gazebo_ros_lds_lfcd_controller" filename="libgazebo_ros_laser.so">
+				  <topicName>scan</topicName>
+				  <frameName>base_scan</frameName>
+				</plugin>
+			</sensor>
+	  </gazebo>
+  </xacro:if>
+	<!-- Ground truth plugin -->
+	<gazebo>
+		<plugin filename="libgazebo_ros_p3d.so" name="gazebo_ros_p3d">
+			<robotNamespace>/</robotNamespace>
+		 	<bodyName>base_link</bodyName>
+			<topicName>ground_truth</topicName>
+			<frameName>world</frameName>
+			<xyzOffsets>0 0 0</xyzOffsets>
+			<rpyOffsets>0 0 0</rpyOffsets>
+			<gaussianNoise>0</gaussianNoise>
+			<alwaysOn>true</alwaysOn>
+		  <updateRate>100</updateRate>
+		</plugin>
+	</gazebo>
   <!-- Gazebo plugin for ROS Control -->
   <gazebo>

File: gpg_description/urdf/gpg.urdf.xacro (robot description, xacro)
@@ -3,10 +3,12 @@
   <xacro:include filename="$(find gpg_description)/urdf/common_properties.xacro"/>
   <xacro:include filename="$(find gpg_description)/urdf/gpg.gazebo.xacro"/>
+  	<xacro:include filename="$(find gpg_description)/urdf/d435/d435.urdf.xacro"/>
   <xacro:property name="CADscale" value="0.0012" />
   <!-- Which sensors to include -->
-  <xacro:arg name="imu"        default="false" />
+  <xacro:arg name="imu"        default="false"/>
+  <xacro:arg name="laser"      default="false"/>
+  <xacro:arg name="d435"       default="false"/>
   <xacro:arg name="distance"   default="false"/>
-  <xacro:arg name="lds"        default="false"/>
-  <!-- ============ 'base_footprint' is the ground link ===================== -->
+<!-- ============ 'base_footprint' is the ground link ===================== -->
   <link name="base_footprint"/>
   <joint name="base_joint" type="fixed">
@@ -16,5 +18,5 @@
     <origin xyz="0 0 0.075" rpy="0 0 0"/>
   </joint>
-  <!-- ============ 'base_link' simulates GoPiGo3 body mass and moment of inertia and act as the robot reference frame =================== -->
+<!-- ============ 'base_link' simulates GoPiGo3 body mass and moment of inertia and act as the robot reference frame =================== -->
   <link name="base_link">
   <!-- **** 'base_link' COLLISION & INERTIA **** -->
@@ -276,6 +278,12 @@
     </link>
   </xacro:macro>
-  <xacro:if value="$(arg lds)">
+  <xacro:if value="$(arg laser)">
     <xacro:lds_sensor/>
   </xacro:if>
+<!-- ============ Realsense Camera d435 ======================== -->
+	<xacro:if value="$(arg d435)">
+		<xacro:sensor_d435 name="d435" topics_ns="d435" parent="base_link" use_nominal_extrinsics="true" simulation="true">
+		  <origin xyz="0.056 0.0 0.06" rpy="0 0 0"/>
+		</xacro:sensor_d435>
+  </xacro:if>
 </robot>
